Commit message: Completed 10 body trials and saved data -EM

File: body_1.urdf (robot description, URDF)
Before this commit: robot robot, 5 links, 4 joints
Links:
- link Body: geometry collision box size=3.00553918342309 0.17536607627353484 4.616851974203088; visual box size=3.00553918342309 0.17536607627353484 4.616851974203088
- link Leg1: geometry collision box size=4.832497300406195 1.4109716076273227 2.6348577614141004; visual box size=4.832497300406195 1.4109716076273227 2.6348577614141004
- link Leg2: geometry collision box size=3.6198084015842147 2.6621521280467455 4.170433918607984; visual box size=3.6198084015842147 2.6621521280467455 4.170433918607984
- link Leg3: geometry collision box size=3.2069690427034026 1.4042026768321025 3.988515854664296; visual box size=3.2069690427034026 1.4042026768321025 3.988515854664296
- link Leg4: geometry collision box size=3.421809631357892 4.4423221427206165 2.4833524629590498; visual box size=3.421809631357892 4.4423221427206165 2.4833524629590498
Joints:
- joint Body_Leg1: origin xyz=-1.2614616511238588 -0.7150865497459549 4.204821157266449 rpy=0 0 0 -> xyz=-1.502769591711545 -0.08768303813676742 4.170433918607984 rpy=0 0 0
- joint Body_Leg2: origin xyz=1.2614616511238588 -0.7150865497459549 4.204821157266449 rpy=0 0 0 -> xyz=1.502769591711545 -0.08768303813676742 4.170433918607984 rpy=0 0 0
- joint Body_Leg3: origin xyz=1.2614616511238588 0.7150865497459549 4.204821157266449 rpy=0 0 0 -> xyz=1.502769591711545 0.08768303813676742 4.170433918607984 rpy=0 0 0
- joint Body_Leg4: origin xyz=-1.2614616511238588 0.7150865497459549 4.204821157266449 rpy=0 0 0 -> xyz=-1.502769591711545 0.08768303813676742 4.170433918607984 rpy=0 0 0

File: body_13.urdf (robot description, URDF)
Before this commit: robot robot, 5 links, 4 joints
Links:
- link Body: geometry collision box size=3.155816142594244 0.17536607627353484 4.616851974203088; visual box size=3.155816142594244 0.17536607627353484 4.616851974203088
Joints:
- joint Body_Leg1: origin xyz=-1.502769591711545 -0.08768303813676742 4.170433918607984 rpy=0 0 0 -> xyz=-1.577908071297122 -0.08768303813676742 4.170433918607984 rpy=0 0 0
- joint Body_Leg2: origin xyz=1.502769591711545 -0.08768303813676742 4.170433918607984 rpy=0 0 0 -> xyz=1.577908071297122 -0.08768303813676742 4.170433918607984 rpy=0 0 0
- joint Body_Leg3: origin xyz=1.502769591711545 0.08768303813676742 4.170433918607984 rpy=0 0 0 -> xyz=1.577908071297122 0.08768303813676742 4.170433918607984 rpy=0 0 0
- joint Body_Leg4: origin xyz=-1.502769591711545 0.08768303813676742 4.170433918607984 rpy=0 0 0 -> xyz=-1.577908071297122 0.08768303813676742 4.170433918607984 rpy=0 0 0

File: body_2.urdf (robot description, URDF)
Before this commit: robot robot, 5 links, 4 joints
Links:
- link Body: geometry collision box size=3.00553918342309 0.17536607627353484 4.616851974203088; visual box size=3.00553918342309 0.17536607627353484 4.616851974203088
- link Leg1: geometry collision box size=4.832497300406195 1.4109716076273227 2.6348577614141004; visual box size=4.832497300406195 1.4109716076273227 2.6348577614141004
- link Leg2: geometry collision box size=3.6198084015842147 2.6621521280467455 4.170433918607984; visual box size=3.6198084015842147 2.6621521280467455 4.170433918607984
- link Leg3: geometry collision box size=3.2069690427034026 1.4042026768321025 3.988515854664296; visual box size=3.2069690427034026 1.4042026768321025 3.988515854664296
- link Leg4: geometry collision box size=3.421809631357892 4.4423221427206165 2.4833524629590498; visual box size=3.421809631357892 4.4423221427206165 2.4833524629590498
Joints:
- joint Body_Leg1: origin xyz=-1.2614616511238588 -0.7150865497459549 4.204821157266449 rpy=0 0 0 -> xyz=-1.502769591711545 -0.08768303813676742 4.170433918607984 rpy=0 0 0
- joint Body_Leg2: origin xyz=1.2614616511238588 -0.7150865497459549 4.204821157266449 rpy=0 0 0 -> xyz=1.502769591711545 -0.08768303813676742 4.170433918607984 rpy=0 0 0
- joint Body_Leg3: origin xyz=1.2614616511238588 0.7150865497459549 4.204821157266449 rpy=0 0 0 -> xyz=1.502769591711545 0.08768303813676742 4.170433918607984 rpy=0 0 0
- joint Body_Leg4: origin xyz=-1.2614616511238588 0.7150865497459549 4.204821157266449 rpy=0 0 0 -> xyz=-1.502769591711545 0.08768303813676742 4.170433918607984 rpy=0 0 0

File: body_3.urdf (robot description, URDF)
Before this commit: robot robot, 5 links, 4 joints
Links:
- link Body: geometry collision box size=3.00553918342309 0.17536607627353484 4.616851974203088; visual box size=3.00553918342309 0.17536607627353484 4.616851974203088
- link Leg1: geometry collision box size=4.832497300406195 1.4109716076273227 2.6348577614141004; visual box size=4.832497300406195 1.4109716076273227 2.6348577614141004
- link Leg2: geometry collision box size=3.6198084015842147 2.6621521280467455 4.170433918607984; visual box size=3.6198084015842147 2.6621521280467455 4.170433918607984
- link Leg3: geometry collision box size=3.2069690427034026 1.4042026768321025 3.988515854664296; visual box size=3.2069690427034026 1.4042026768321025 3.988515854664296
- link Leg4: geometry collision box size=3.421809631357892 4.4423221427206165 2.4833524629590498; visual box size=3.421809631357892 4.4423221427206165 2.4833524629590498
Joints:
- joint Body_Leg1: origin xyz=-1.0210680993891208 -0.7150865497459549 4.204821157266449 rpy=0 0 0 -> xyz=-1.502769591711545 -0.08768303813676742 4.170433918607984 rpy=0 0 0
- joint Body_Leg2: origin xyz=1.0210680993891208 -0.7150865497459549 4.204821157266449 rpy=0 0 0 -> xyz=1.502769591711545 -0.08768303813676742 4.170433918607984 rpy=0 0 0
- joint Body_Leg3: origin xyz=1.0210680993891208 0.7150865497459549 4.204821157266449 rpy=0 0 0 -> xyz=1.502769591711545 0.08768303813676742 4.170433918607984 rpy=0 0 0
- joint Body_Leg4: origin xyz=-1.0210680993891208 0.7150865497459549 4.204821157266449 rpy=0 0 0 -> xyz=-1.502769591711545 0.08768303813676742 4.170433918607984 rpy=0 0 0

File: body_5.urdf (robot description, URDF)
Before this commit: robot robot, 5 links, 4 joints
Links:
- link Body: geometry collision box size=3.00553918342309 0.17536607627353484 4.616851974203088; visual box size=3.00553918342309 0.17536607627353484 4.616851974203088
- link Leg1: geometry collision box size=4.832497300406195 1.4109716076273227 2.6348577614141004; visual box size=4.832497300406195 1.4109716076273227 2.6348577614141004
- link Leg2: geometry collision box size=3.6198084015842147 2.6621521280467455 4.170433918607984; visual box size=3.6198084015842147 2.6621521280467455 4.170433918607984
- link Leg3: geometry collision box size=3.2069690427034026 1.4042026768321025 3.988515854664296; visual box size=3.2069690427034026 1.4042026768321025 3.988515854664296
- link Leg4: geometry collision box size=3.421809631357892 4.4423221427206165 2.4833524629590498; visual box size=3.421809631357892 4.4423221427206165 2.4833524629590498
Joints:
- joint Body_Leg1: origin xyz=-2.0700012750297154 -1.5418840920243104 4.350284275227032 rpy=0 0 0 -> xyz=-1.502769591711545 -0.08768303813676742 4.170433918607984 rpy=0 0 0
- joint Body_Leg2: origin xyz=2.0700012750297154 -1.5418840920243104 4.350284275227032 rpy=0 0 0 -> xyz=1.502769591711545 -0.08768303813676742 4.170433918607984 rpy=0 0 0
- joint Body_Leg3: origin xyz=2.0700012750297154 1.5418840920243104 4.350284275227032 rpy=0 0 0 -> xyz=1.502769591711545 0.08768303813676742 4.170433918607984 rpy=0 0 0
- joint Body_Leg4: origin xyz=-2.0700012750297154 1.5418840920243104 4.350284275227032 rpy=0 0 0 -> xyz=-1.502769591711545 0.08768303813676742 4.170433918607984 rpy=0 0 0

File: body_6.urdf (robot description, URDF)
Before this commit: robot robot, 5 links, 4 joints
Links:
- link Body: geometry collision box size=3.00553918342309 0.17536607627353484 4.616851974203088; visual box size=3.00553918342309 0.17536607627353484 4.616851974203088
- link Leg1: geometry collision box size=4.832497300406195 1.4109716076273227 2.6348577614141004; visual box size=4.832497300406195 1.4109716076273227 2.6348577614141004
- link Leg2: geometry collision box size=3.6198084015842147 2.6621521280467455 4.170433918607984; visual box size=3.6198084015842147 2.6621521280467455 4.170433918607984
- link Leg3: geometry collision box size=3.2069690427034026 1.4042026768321025 3.988515854664296; visual box size=3.2069690427034026 1.4042026768321025 3.988515854664296
- link Leg4: geometry collision box size=3.421809631357892 4.4423221427206165 2.4833524629590498; visual box size=3.421809631357892 4.4423221427206165 2.4833524629590498
Joints:
- joint Body_Leg1: origin xyz=-0.8429525462503709 -1.0168564911154097 2.0692480457536435 rpy=0 0 0 -> xyz=-1.502769591711545 -0.08768303813676742 4.170433918607984 rpy=0 0 0
- joint Body_Leg2: origin xyz=0.8429525462503709 -1.0168564911154097 2.0692480457536435 rpy=0 0 0 -> xyz=1.502769591711545 -0.08768303813676742 4.170433918607984 rpy=0 0 0
- joint Body_Leg3: origin xyz=0.8429525462503709 1.0168564911154097 2.0692480457536435 rpy=0 0 0 -> xyz=1.502769591711545 0.08768303813676742 4.170433918607984 rpy=0 0 0
- joint Body_Leg4: origin xyz=-0.8429525462503709 1.0168564911154097 2.0692480457536435 rpy=0 0 0 -> xyz=-1.502769591711545 0.08768303813676742 4.170433918607984 rpy=0 0 0

File: body_7.urdf (robot description, URDF)
Before this commit: robot robot, 5 links, 4 joints
Links:
- link Body: geometry collision box size=3.00553918342309 0.17536607627353484 4.616851974203088; visual box size=3.00553918342309 0.17536607627353484 4.616851974203088
- link Leg1: geometry collision box size=4.832497300406195 1.4109716076273227 2.6348577614141004; visual box size=4.832497300406195 1.4109716076273227 2.6348577614141004
- link Leg2: geometry collision box size=3.6198084015842147 2.6621521280467455 4.170433918607984; visual box size=3.6198084015842147 2.6621521280467455 4.170433918607984
- link Leg3: geometry collision box size=3.2069690427034026 1.4042026768321025 3.988515854664296; visual box size=3.2069690427034026 1.4042026768321025 3.988515854664296
- link Leg4: geometry collision box size=3.421809631357892 4.4423221427206165 2.4833524629590498; visual box size=3.421809631357892 4.4423221427206165 2.4833524629590498
Joints:
- joint Body_Leg1: origin xyz=-1.8934328033192664 -2.05951725748372 4.448067351649415 rpy=0 0 0 -> xyz=-1.502769591711545 -0.08768303813676742 4.170433918607984 rpy=0 0 0
- joint Body_Leg2: origin xyz=1.8934328033192664 -2.05951725748372 4.448067351649415 rpy=0 0 0 -> xyz=1.502769591711545 -0.08768303813676742 4.170433918607984 rpy=0 0 0
- joint Body_Leg3: origin xyz=1.8934328033192664 2.05951725748372 4.448067351649415 rpy=0 0 0 -> xyz=1.502769591711545 0.08768303813676742 4.170433918607984 rpy=0 0 0
- joint Body_Leg4: origin xyz=-1.8934328033192664 2.05951725748372 4.448067351649415 rpy=0 0 0 -> xyz=-1.502769591711545 0.08768303813676742 4.170433918607984 rpy=0 0 0

File: body_8.urdf (robot description, URDF)
Before this commit: robot robot, 5 links, 4 joints
Links:
- link Body: geometry collision box size=3.00553918342309 0.17536607627353484 4.616851974203088; visual box size=3.00553918342309 0.17536607627353484 4.616851974203088
- link Leg1: geometry collision box size=4.832497300406195 1.4109716076273227 2.6348577614141004; visual box size=4.832497300406195 1.4109716076273227 2.6348577614141004
- link Leg2: geometry collision box size=3.6198084015842147 2.6621521280467455 4.170433918607984; visual box size=3.6198084015842147 2.6621521280467455 4.170433918607984
- link Leg3: geometry collision box size=3.2069690427034026 1.4042026768321025 3.988515854664296; visual box size=3.2069690427034026 1.4042026768321025 3.988515854664296
- link Leg4: geometry collision box size=3.421809631357892 4.4423221427206165 2.4833524629590498; visual box size=3.421809631357892 4.4423221427206165 2.4833524629590498
Joints:
- joint Body_Leg1: origin xyz=-0.8663744235098253 -0.4016926346582869 3.2977000426962944 rpy=0 0 0 -> xyz=-1.502769591711545 -0.08768303813676742 4.170433918607984 rpy=0 0 0
- joint Body_Leg2: origin xyz=0.8663744235098253 -0.4016926346582869 3.2977000426962944 rpy=0 0 0 -> xyz=1.502769591711545 -0.08768303813676742 4.170433918607984 rpy=0 0 0
- joint Body_Leg3: origin xyz=0.8663744235098253 0.4016926346582869 3.2977000426962944 rpy=0 0 0 -> xyz=1.502769591711545 0.08768303813676742 4.170433918607984 rpy=0 0 0
- joint Body_Leg4: origin xyz=-0.8663744235098253 0.4016926346582869 3.2977000426962944 rpy=0 0 0 -> xyz=-1.502769591711545 0.08768303813676742 4.170433918607984 rpy=0 0 0

File: body_9.urdf (robot description, URDF)
Before this commit: robot robot, 5 links, 4 joints
Links:
- link Body: geometry collision box size=3.00553918342309 0.17536607627353484 4.616851974203088; visual box size=3.00553918342309 0.17536607627353484 4.616851974203088
- link Leg1: geometry collision box size=4.832497300406195 1.4109716076273227 2.6348577614141004; visual box size=4.832497300406195 1.4109716076273227 2.6348577614141004
- link Leg2: geometry collision box size=3.6198084015842147 2.6621521280467455 4.170433918607984; visual box size=3.6198084015842147 2.6621521280467455 4.170433918607984
- link Leg3: geometry collision box size=3.2069690427034026 1.4042026768321025 3.988515854664296; visual box size=3.2069690427034026 1.4042026768321025 3.988515854664296
- link Leg4: geometry collision box size=3.421809631357892 4.4423221427206165 2.4833524629590498; visual box size=3.421809631357892 4.4423221427206165 2.4833524629590498
Joints:
- joint Body_Leg1: origin xyz=-0.18509262181390623 -0.0023695225861705693 3.9714896757854734 rpy=0 0 0 -> xyz=-1.502769591711545 -0.08768303813676742 4.170433918607984 rpy=0 0 0
- joint Body_Leg2: origin xyz=0.18509262181390623 -0.0023695225861705693 3.9714896757854734 rpy=0 0 0 -> xyz=1.502769591711545 -0.08768303813676742 4.170433918607984 rpy=0 0 0
- joint Body_Leg3: origin xyz=0.18509262181390623 0.0023695225861705693 3.9714896757854734 rpy=0 0 0 -> xyz=1.502769591711545 0.08768303813676742 4.170433918607984 rpy=0 0 0
- joint Body_Leg4: origin xyz=-0.18509262181390623 0.0023695225861705693 3.9714896757854734 rpy=0 0 0 -> xyz=-1.502769591711545 0.08768303813676742 4.170433918607984 rpy=0 0 0
